File: GamePad/GamePad.kicad_pcb (KiCad board)
At the start: 2 copper layers, 85 x 48 mm, 17 parts, among them J1 Conn_01x04_Socket (bumper), J2 Conn_01x02_Socket (power)

Commit message: added custom pcb
Other:
- board text added: "5V"
- board text added: "Arya's Gamepad!"
- board text added: "GND"
- board text added: "GPIO 1 -> 40"
- board text added: "direction"
- board text added: "xoab"
Changed lines of the file:
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@@
 		(layer "Edge.Cuts")
+	)
+	(gr_text "GPIO 1 -> 40"
+		(at 42.8625 195.2625 0)
+		(layer "F.SilkS")
+		(effects
+			(font
+				(size 1 1)
+				(thickness 0.1)
+			)
+			(justify left bottom)
+		)
+	)
+	(gr_text "GND\n"
+		(at 90.4875 188.11875 90)
+		(layer "F.SilkS")
+		(effects
+			(font
+				(size 1 1)
+				(thickness 0.1)
+			)
+			(justify left bottom)
+		)
+	)
+	(gr_text "GND\n"
+		(at 88.10625 188.11875 90)
+		(layer "F.SilkS")
+		(effects
+			(font
+				(size 1 1)
+				(thickness 0.1)
+			)
+			(justify left bottom)
+		)
+	)
+	(gr_text "GND\n"
+		(at 21.43125 195.2625 0)
+		(layer "F.SilkS")
+		(effects
+			(font
+				(size 1 1)
+				(thickness 0.1)
+			)
+			(justify left bottom)
+		)
+	)
+	(gr_text "direction"
+		(at 21.43125 183.35625 0)
+		(layer "F.SilkS")
+		(effects
+			(font
+				(size 1 1)
+				(thickness 0.1)
+			)
+			(justify left bottom)
+		)
+	)
+	(gr_text "Arya's Gamepad!\n"
+		(at 19.05 154.78125 0)
+		(layer "F.SilkS")
+		(effects
+			(font
+				(size 1 1)
+				(thickness 0.1)
+			)
+			(justify left bottom)
+		)
+	)
+	(gr_text "xoab\n"
+		(at 90.4875 180.975 0)
+		(layer "F.SilkS")
+		(effects
+			(font
+				(size 1 1)
+				(thickness 0.1)
+			)
+			(justify left bottom)
+		)
+	)
+	(gr_text "5V\n"
+		(at 16.66875 195.2625 0)
+		(layer "F.SilkS")
+		(effects
+			(font
+				(size 1 1)
+				(thickness 0.1)
+			)
+			(justify left bottom)
+		)
 	)
 	(segment
