File: GamePad/GamePad_Zero/GamePad_Zero.kicad_pcb (KiCad board)
At the start: 2 copper layers, 150 x 60 mm, 16 parts, among them J1 Conn_02x20_Odd_Even, SW1 SW_SPDT, U1 2465, x1 SW_Push, y1 SW_Push

Commit message: finishing touches
Parts:
- added G***: LOGO, LOGO, F.Cu at (75.0, 31.7)
- added G***: LOGO, LOGO, B.Cu at (21.4, 42.9)
- added G***: LOGO, LOGO, B.Cu at (75.1, 31.6)
Other:
- board text added: "1000C Here"
- board text added: "Designed by Arya Chakrabarti"
- board text added: "GamePAD"
- board text added: "GamePAD v2"
- board text added: "Spherical Cow Production Co."
- board text added: "finished 6/30/25"
